Commit message: Fixed the setup file
- Fixed the issue about mesh import
- Removed the inertial components in the URDF

File: urdf/a0509.blue.urdf (robot description, URDF)
Before this commit: robot doosan_a0509, 8 links, 7 joints
Joints:
- joint elbow_joint: limit lower=-1.57 upper=1.57 effort=0 velocity=0.5 -> lower=-2.617 upper=2.617 effort=30 velocity=1.571
- joint end_effector_joint: limit lower=-1.57 upper=1.57 effort=0 velocity=0.5 -> lower=-2.617 upper=2.617 effort=30 velocity=1.571
- joint shoulder_joint: limit lower=-1.57 upper=1.57 effort=0 velocity=0.5 -> lower=-2.617 upper=2.617 effort=30 velocity=1.571
- joint wrist_pitch_joint: limit lower=-1.57 upper=1.57 effort=0 velocity=0.5 -> lower=-2.617 upper=2.617 effort=30 velocity=1.571
- joint wrist_roll_joint: limit lower=-1.57 upper=1.57 effort=0 velocity=0.5 -> lower=-2.617 upper=2.617 effort=30 velocity=1.571
- joint wrist_yaw_joint: limit lower=-1.57 upper=1.57 effort=0 velocity=0.5 -> lower=-2.617 upper=2.617 effort=30 velocity=1.571

Commit message: Added the inertial parameters

File: urdf/a0509.blue.urdf (robot description, URDF)
Before this commit: robot doosan_a0509, 8 links, 7 joints
Links:
- link base_link: mass None -> 3.722
- link elbow_link: mass None -> 10.569
- link end_effector_link: mass None -> 1.128
- link shoulder_link: mass None -> 7.446
- link wrist_pitch_link: mass None -> 3.614
- link wrist_roll_link: mass None -> 3.785
- link wrist_yaw_link: mass None -> 2.598

Commit message: Updated the package uri for meshes
- Earlier it was referring from the package "robot_arm"
- Fixed all occurences so now it refers from the package://dsr_a0509_description

File: urdf/a0509.blue.urdf (robot description, URDF)
Before this commit: robot doosan_a0509, 8 links, 7 joints
Links:
- link base_link: geometry visual mesh filename=package://dsr_a0509_description/meshes/A0509_0_0.dae scale=0.001 0.001 0.001
- link elbow_link: geometry visual mesh filename=package://dsr_a0509_description/meshes/A0509_2_0.dae scale=0.001 0.001 0.001; visual mesh filename=package://dsr_a0509_description/meshes/A0509_2_1.dae scale=0.001 0.001 0.001
- link end_effector_link: geometry visual mesh filename=package://dsr_a0509_description/meshes/A0509_6_0.dae scale=0.001 0.001 0.001
- link shoulder_link: geometry visual mesh filename=package://dsr_a0509_description/meshes/A0509_1_0.dae scale=0.001 0.001 0.001; visual mesh filename=package://dsr_a0509_description/meshes/A0509_1_1.dae scale=0.001 0.001 0.001
- link wrist_pitch_link: geometry visual mesh filename=package://dsr_a0509_description/meshes/A0509_3_0.dae scale=0.001 0.001 0.001; visual mesh filename=package://dsr_a0509_description/meshes/A0509_3_1.dae scale=0.001 0.001 0.001
- link wrist_roll_link: geometry visual mesh filename=package://dsr_a0509_description/meshes/A0509_4_0.dae scale=0.001 0.001 0.001; visual mesh filename=package://dsr_a0509_description/meshes/A0509_4_1.dae scale=0.001 0.001 0.001
- link wrist_yaw_link: geometry visual mesh filename=package://dsr_a0509_description/meshes/A0509_5_0.dae scale=0.001 0.001 0.001; visual mesh filename=package://dsr_a0509_description/meshes/A0509_5_1.dae scale=0.001 0.001 0.001

Commit message: Added collision meshes

File: urdf/a0509.blue.urdf (robot description, URDF)
Before this commit: robot doosan_a0509, 8 links, 7 joints
Links:
- link base_link: geometry collision mesh filename=package://dsr_a0509_description/meshes/A0509_0_0.dae scale=0.001 0.001 0.001; visual mesh filename=package://dsr_a0509_description/meshes/A0509_0_0.dae scale=0.001 0.001 0.001
- link elbow_link: geometry collision mesh filename=package://dsr_a0509_description/meshes/A0509_2_0.dae scale=0.001 0.001 0.001; collision mesh filename=package://dsr_a0509_description/meshes/A0509_2_1.dae scale=0.001 0.001 0.001
- link end_effector_link: geometry collision mesh filename=package://dsr_a0509_description/meshes/A0509_6_0.dae scale=0.001 0.001 0.001; visual mesh filename=package://dsr_a0509_description/meshes/A0509_6_0.dae scale=0.001 0.001 0.001
- link shoulder_link: geometry collision mesh filename=package://dsr_a0509_description/meshes/A0509_1_0.dae scale=0.001 0.001 0.001; collision mesh filename=package://dsr_a0509_description/meshes/A0509_1_1.dae scale=0.001 0.001 0.001
- link wrist_pitch_link: geometry collision mesh filename=package://dsr_a0509_description/meshes/A0509_3_0.dae scale=0.001 0.001 0.001; collision mesh filename=package://dsr_a0509_description/meshes/A0509_3_1.dae scale=0.001 0.001 0.001
- link wrist_roll_link: geometry collision mesh filename=package://dsr_a0509_description/meshes/A0509_4_0.dae scale=0.001 0.001 0.001; collision mesh filename=package://dsr_a0509_description/meshes/A0509_4_1.dae scale=0.001 0.001 0.001
- link wrist_yaw_link: geometry collision mesh filename=package://dsr_a0509_description/meshes/A0509_5_0.dae scale=0.001 0.001 0.001; collision mesh filename=package://dsr_a0509_description/meshes/A0509_5_1.dae scale=0.001 0.001 0.001
